File: rev.03/MM-control.sch (KiCad schematic (older format))
At the start: 86 parts, among them J1 MX-105017-0001, P1 MOLEX 70543-0004, P11 MP, P12 MP, P2 MOLEX 70543-0003, P3 MP, P4 MOLEX 70543-0002, P5 ICSP, P6 ShiftOut, P7 MOLEX 70543-0004, U2 74HC595, U4 ATmega32U4, U8 ATmega32U4, U9 74HC595, Y1 LFXTAL035264BULK 16MHz

Commit message: Update files that KiCAD modified. Update BOM.
Parts:
- C1, C10, C2, C3, C4, C6, C60, C9: symbol device:C -> MM-control-rescue:C-device
- C59: symbol device:CP_Small -> MM-control-rescue:CP_Small-device
- D1, D6, D7: symbol device:D_ALT -> MM-control-rescue:D_ALT-device
- D14, D15, D16, D17, D18, D19, D20, D21, D22, D23: symbol device:LED_Small_ALT -> MM-control-rescue:LED_Small_ALT-device
- D8, D9: symbol device:LED_ALT -> MM-control-rescue:LED_ALT-device
- F1, F2: symbol device:Polyfuse_Small -> MM-control-rescue:Polyfuse_Small-device
- J1: symbol ok1hra:USB-micro -> MM-control-rescue:USB-micro-ok1hra
- L1, L2, L21, L22, L3, L5, L6, L7: symbol device:L_Core_Ferrite_Small -> MM-control-rescue:L_Core_Ferrite_Small-device
- P1, P6: symbol conn:CONN_01X05 -> MM-control-rescue:CONN_01X05-conn
- P11, P12, P3: symbol conn:CONN_01X01 -> MM-control-rescue:CONN_01X01-conn
- P2: symbol conn:CONN_02X02 -> MM-control-rescue:CONN_02X02-conn
- P4: symbol conn:CONN_01X03 -> MM-control-rescue:CONN_01X03-conn
- P7: symbol conn:CONN_01X06 -> MM-control-rescue:CONN_01X06-conn
- R1, R10, R11, R12, R13, R15, R16, R17, R18, R2, R21, R22, R23, R24, R25, R38, R39, R4, R40, R41, R42, R43, R44, R45, R46, R5, R6, R7, R8, R9: symbol device:R -> MM-control-rescue:R-device
- S1, S2, S3, S4: symbol ok1hra:TACT-SW2 -> MM-control-rescue:TACT-SW2-ok1hra
- U2, U9: symbol ok1hra:74HC595 -> MM-control-rescue:74HC595-ok1hra
- U4, U8: symbol atmel:ATmega32U4 -> MM-control-rescue:ATmega32U4-atmel
- Y1: symbol device:Crystal_GND24 -> MM-control-rescue:Crystal_GND24-device
