File: rev.03/trinamic.sch (KiCad schematic (older format))
At the start: 78 parts, among them P10 MOLEX 70543-0003, P8 MOLEX 70543-0003, P9 MOLEX 70543-0003, U5 TMC2130-LA, U6 TMC2130-LA, U7 TMC2130-LA

Commit message: Update files that KiCAD modified. Update BOM.
Parts:
- C12, C13, C14, C15, C16, C17, C18, C19, C20, C21, C22, C23, C24, C25, C26, C27, C28, C29, C32, C33, C34, C35, C36, C37, C38, C39, C40, C41, C42, C44, C45, C46, C47, C48, C49, C50, C51, C52, C54, C55, C56, C57, C58: symbol device:C_Small -> MM-control-rescue:C_Small-device
- C30, C31, C43, C53: symbol device:CP_Small -> MM-control-rescue:CP_Small-device
- L10, L11, L12, L13, L14, L15, L16, L17, L18, L19, L20, L8, L9: symbol device:L_Core_Ferrite_Small -> MM-control-rescue:L_Core_Ferrite_Small-device
- P10, P8, P9: symbol conn:CONN_01X04 -> MM-control-rescue:CONN_01X04-conn
- R26, R27, R28, R29, R30, R31, R32, R33, R34, R35, R36, R37: symbol device:R -> MM-control-rescue:R-device
- U5, U6, U7: symbol ok1hra:TCM2130-LA -> MM-control-rescue:TCM2130-LA-ok1hra
